File: PCB/Hexapod PCB KiCad Project/Leg.kicad_sch (KiCad schematic)
At the start: 3 parts, among them J1 Conn_01x03, J3 Conn_01x03, J4 Conn_01x03

Commit message: traces
Changed lines of the file:
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@@
   (symbol (lib_id "Connector_Generic:Conn_01x03") (at 157.48 112.395 0) (unit 1)
     (in_bom yes) (on_board yes) (dnp no) (fields_autoplaced)
-    (property "Reference" "J4" (at 160.655 111.125 0)
+    (property "Reference" "J4" (at 160.02 111.125 0)
       (effects (font (size 1.27 1.27)) (justify left))
     )
-    (property "Value" "Conn_01x03" (at 160.655 113.665 0)
+    (property "Value" "Conn_01x03" (at 160.02 113.665 0)
       (effects (font (size 1.27 1.27)) (justify left))
     )
@@
         )
         (path "/55308d4e-8005-4344-88fa-e9149757c1fd/50b45e52-3dc5-4b44-ac76-89d0a21a0c01"
-          (reference "J4") (unit 1)
+          (reference "Tib6") (unit 1)
         )
         (path "/55308d4e-8005-4344-88fa-e9149757c1fd/ecec22b4-9708-4564-b944-a2a2a8ec580f"
-          (reference "J8") (unit 1)
+          (reference "Tib5") (unit 1)
         )
         (path "/55308d4e-8005-4344-88fa-e9149757c1fd/64ba9eee-1de7-4ed5-809f-3e6bab105923"
-          (reference "J11") (unit 1)
+          (reference "Tib4") (unit 1)
         )
         (path "/55308d4e-8005-4344-88fa-e9149757c1fd/9008ff35-f48d-43a0-8ef3-d1c49a9cb0c0"
-          (reference "J14") (unit 1)
+          (reference "Tib3") (unit 1)
         )
         (path "/55308d4e-8005-4344-88fa-e9149757c1fd/059d42e5-5a73-4bd5-a346-feb4dd2c71e4"
-          (reference "J17") (unit 1)
+          (reference "Tib2") (unit 1)
         )
         (path "/55308d4e-8005-4344-88fa-e9149757c1fd/efed6682-a9f2-4b0f-80cc-97ecacc1acb6"
-          (reference "J20") (unit 1)
+          (reference "Tib1") (unit 1)
         )
       )
@@
   (symbol (lib_id "Connector_Generic:Conn_01x03") (at 157.48 99.06 0) (unit 1)
     (in_bom yes) (on_board yes) (dnp no) (fields_autoplaced)
-    (property "Reference" "J3" (at 160.655 97.79 0)
+    (property "Reference" "J3" (at 160.02 97.79 0)
       (effects (font (size 1.27 1.27)) (justify left))
     )
-    (property "Value" "Conn_01x03" (at 160.655 100.33 0)
+    (property "Value" "Conn_01x03" (at 160.02 100.33 0)
       (effects (font (size 1.27 1.27)) (justify left))
     )
@@
         )
         (path "/55308d4e-8005-4344-88fa-e9149757c1fd/50b45e52-3dc5-4b44-ac76-89d0a21a0c01"
-          (reference "J3") (unit 1)
+          (reference "Fem6") (unit 1)
         )
         (path "/55308d4e-8005-4344-88fa-e9149757c1fd/ecec22b4-9708-4564-b944-a2a2a8ec580f"
-          (reference "J7") (unit 1)
+          (reference "Fem5") (unit 1)
         )
         (path "/55308d4e-8005-4344-88fa-e9149757c1fd/64ba9eee-1de7-4ed5-809f-3e6bab105923"
-          (reference "J10") (unit 1)
+          (reference "Fem4") (unit 1)
         )
         (path "/55308d4e-8005-4344-88fa-e9149757c1fd/9008ff35-f48d-43a0-8ef3-d1c49a9cb0c0"
-          (reference "J13") (unit 1)
+          (reference "Fem3") (unit 1)
         )
         (path "/55308d4e-8005-4344-88fa-e9149757c1fd/059d42e5-5a73-4bd5-a346-feb4dd2c71e4"
-          (reference "J16") (unit 1)
+          (reference "Fem2") (unit 1)
         )
         (path "/55308d4e-8005-4344-88fa-e9149757c1fd/efed6682-a9f2-4b0f-80cc-97ecacc1acb6"
-          (reference "J19") (unit 1)
+          (reference "Fem1") (unit 1)
         )
       )
@@
   (symbol (lib_id "Connector_Generic:Conn_01x03") (at 157.48 86.995 0) (unit 1)
     (in_bom yes) (on_board yes) (dnp no) (fields_autoplaced)
-    (property "Reference" "J1" (at 160.655 85.725 0)
+    (property "Reference" "J1" (at 160.02 85.725 0)
       (effects (font (size 1.27 1.27)) (justify left))
     )
-    (property "Value" "Conn_01x03" (at 160.655 88.265 0)
+    (property "Value" "Conn_01x03" (at 160.02 88.265 0)
       (effects (font (size 1.27 1.27)) (justify left))
     )
@@
         )
         (path "/55308d4e-8005-4344-88fa-e9149757c1fd/50b45e52-3dc5-4b44-ac76-89d0a21a0c01"
-          (reference "J1") (unit 1)
+          (reference "Cox6") (unit 1)
         )
         (path "/55308d4e-8005-4344-88fa-e9149757c1fd/ecec22b4-9708-4564-b944-a2a2a8ec580f"
-          (reference "J6") (unit 1)
+          (reference "Cox5") (unit 1)
         )
         (path "/55308d4e-8005-4344-88fa-e9149757c1fd/64ba9eee-1de7-4ed5-809f-3e6bab105923"
-          (reference "J9") (unit 1)
+          (reference "Cox4") (unit 1)
         )
         (path "/55308d4e-8005-4344-88fa-e9149757c1fd/9008ff35-f48d-43a0-8ef3-d1c49a9cb0c0"
-          (reference "J12") (unit 1)
+          (reference "Cox3") (unit 1)
         )
         (path "/55308d4e-8005-4344-88fa-e9149757c1fd/059d42e5-5a73-4bd5-a346-feb4dd2c71e4"
-          (reference "J15") (unit 1)
+          (reference "Cox2") (unit 1)
         )
         (path "/55308d4e-8005-4344-88fa-e9149757c1fd/efed6682-a9f2-4b0f-80cc-97ecacc1acb6"
-          (reference "J18") (unit 1)
+          (reference "Cox1") (unit 1)
         )
       )
