File: PCB/Hexapod PCB KiCad Project/Hexapod PCB KiCad Project.kicad_pcb (KiCad board)
At the start: 2 copper layers, 1 part, among them IC1 TEENSY_4.1

Commit message: pcb updates
Parts:
- removed IC1: TEENSY_4.1, TEENSY_4.1:TEENSY41
- added J1: Male Pin Header 1x3, Connector_PinHeader_2.54mm:PinHeader_1x03_P2.54mm_Vertical, F.Cu at (127.0, 69.6)
- added J2: Power Terminal, Terminal 2 Pin:CUI_TB005-762-02BE, F.Cu at (83.8, 101.5)
- added U1: DEV-16771, TEENSY 4.1:MODULE_DEV-16771, F.Cu at (151.6, 98.0)

Commit message: Pcb updates
Parts:
- added C1: 50V 10uF, Capacitor_THT:CP_Radial_D5.0mm_P2.00mm, F.Cu at (139.0, 73.7)
- added C2: 50V 0.1uF, Capacitor_THT:CP_Radial_D4.0mm_P2.00mm, F.Cu at (139.0, 68.6)
- added C3: 16V 1000uf, Capacitor_THT:CP_Radial_D10.0mm_P5.00mm, F.Cu at (119.6, 111.8)
- added C4: 16V 1000uf, Capacitor_THT:CP_Radial_D10.0mm_P5.00mm, F.Cu at (120.8, 92.7)
- added H1: MountingHole, MountingHole:MountingHole_3.2mm_M3, F.Cu at (107.9, 77.7)
- added H2: MountingHole, MountingHole:MountingHole_3.2mm_M3, F.Cu at (179.1, 77.7)
- added H3: MountingHole, MountingHole:MountingHole_3.2mm_M3, F.Cu at (107.9, 125.7)
- added H4: MountingHole, MountingHole:MountingHole_3.2mm_M3, F.Cu at (179.1, 125.7)
- added J10: Conn_01x03, Connector_PinHeader_2.54mm:PinHeader_1x03_P2.54mm_Vertical, B.Cu at (127.8, 142.3)
- added J11: Conn_01x03, Connector_PinHeader_2.54mm:PinHeader_1x03_P2.54mm_Vertical, B.Cu at (123.2, 142.3)
- added J12: Conn_01x03, Connector_PinHeader_2.54mm:PinHeader_1x03_P2.54mm_Vertical, B.Cu at (123.6, 61.0)
- added J13: Conn_01x03, Connector_PinHeader_2.54mm:PinHeader_1x03_P2.54mm_Vertical, B.Cu at (128.3, 61.0)
- added J14: Conn_01x03, Connector_PinHeader_2.54mm:PinHeader_1x03_P2.54mm_Vertical, B.Cu at (132.9, 61.0)
- added J15: Conn_01x03, Connector_PinHeader_2.54mm:PinHeader_1x03_P2.54mm_Vertical, B.Cu at (138.9, 61.0)
- added J16: Conn_01x03, Connector_PinHeader_2.54mm:PinHeader_1x03_P2.54mm_Vertical, B.Cu at (143.5, 61.0)
- added J17: Conn_01x03, Connector_PinHeader_2.54mm:PinHeader_1x03_P2.54mm_Vertical, B.Cu at (148.2, 61.0)
- added J18: Conn_01x03, Connector_PinHeader_2.54mm:PinHeader_1x03_P2.54mm_Vertical, B.Cu at (154.1, 60.9)
- added J19: Conn_01x03, Connector_PinHeader_2.54mm:PinHeader_1x03_P2.54mm_Vertical, B.Cu at (158.8, 60.9)
- added J20: Conn_01x03, Connector_PinHeader_2.54mm:PinHeader_1x03_P2.54mm_Vertical, B.Cu at (163.4, 60.9)
- added J3: Conn_01x03, Connector_PinHeader_2.54mm:PinHeader_1x03_P2.54mm_Vertical, B.Cu at (159.2, 142.3)
- added J4: Conn_01x03, Connector_PinHeader_2.54mm:PinHeader_1x03_P2.54mm_Vertical, B.Cu at (154.5, 142.3)
- added J5: Switch, Terminal 2 Pin:CUI_TB005-762-02BE, F.Cu at (110.5, 88.9)
- added J6: Conn_01x03, Connector_PinHeader_2.54mm:PinHeader_1x03_P2.54mm_Vertical, B.Cu at (148.2, 142.2)
- added J7: Conn_01x03, Connector_PinHeader_2.54mm:PinHeader_1x03_P2.54mm_Vertical, B.Cu at (143.5, 142.2)
- added J8: Conn_01x03, Connector_PinHeader_2.54mm:PinHeader_1x03_P2.54mm_Vertical, B.Cu at (138.9, 142.2)
- added J9: Conn_01x03, Connector_PinHeader_2.54mm:PinHeader_1x03_P2.54mm_Vertical, B.Cu at (132.5, 142.3)
- added R1: 10k, Resistor_THT:R_Axial_DIN0207_L6.3mm_D2.5mm_P7.62mm_Horizontal, F.Cu at (130.8, 82.5)
- added R2: 22k, Resistor_THT:R_Axial_DIN0207_L6.3mm_D2.5mm_P7.62mm_Horizontal, F.Cu at (130.8, 86.4)
- added U2: Voltage Regulator, Voltage Regulator LM2596:Voltage Regulator LM2596, F.Cu at (128.7, 113.1)
- added U3: NRF24L01_Breakout, RF_Module:nRF24L01_Breakout, F.Cu at (147.0, 69.3)
- added U4: Gyro, MPU6050 THT:MPU6050 THT, B.Cu at (132.1, 101.9)
- J1: value Male Pin Header 1x3 -> Conn_01x03; moved to B.Cu
- J2: value Power Terminal -> Battery
- U1: footprint TEENSY 4.1:MODULE_DEV-16771 -> Teensy 4.1:MODULE_DEV-16771
- moved J1 81.5 mm to (163.8, 142.3), turned to 180 degrees
- moved J2 27.2 mm to (110.5, 106.7), turned to -90 degrees
- moved U1 8.39 mm to (160.0, 97.8), turned to 180 degrees
Connections:
- net Net-(U1-3.3V-Pad3.3V_1) renamed +3.3V
- J1 pad 1: unconnected-(J1-Pin_1-Pad1) -> GND
- J1 pad 2: unconnected-(J1-Pin_2-Pad2) -> +BATT
- J1 pad 3: unconnected-(J1-Pin_3-Pad3) -> Leg1 Coxa
- J2 pad 1: unconnected-(J2-Pad1) -> GND
- J2 pad 2: unconnected-(J2-Pad2) -> Net-(J2-Pad2)
- U1 pad 10: unconnected-(U1-CS1-Pad10) -> Leg1 Tibia
- U1 pad 11: unconnected-(U1-MOSI-Pad11) -> MOSI
- U1 pad 12: unconnected-(U1-MISO-Pad12) -> MISO
- U1 pad 13: unconnected-(U1-SCK-Pad13) -> SCK
- U1 pad 14: unconnected-(U1-A0-Pad14) -> Leg6 Femur
- U1 pad 15: unconnected-(U1-A1-Pad15) -> Leg6 Coxa
- U1 pad 16: unconnected-(U1-A2-Pad16) -> Battery Voltage Divider
- U1 pad 18: unconnected-(U1-A4-Pad18) -> Gyro SDA
- U1 pad 19: unconnected-(U1-A5-Pad19) -> Gyro SCL
- U1 pad 2: unconnected-(U1-OUT2-Pad2) -> Leg3 Coxa
- U1 pad 24: unconnected-(U1-A10-Pad24) -> Leg4 Tibia
- U1 pad 25: unconnected-(U1-A11-Pad25) -> Leg4 Femur
- U1 pad 26: unconnected-(U1-A12-Pad26) -> CE
- U1 pad 27: unconnected-(U1-A13-Pad27) -> CSN
- U1 pad 28: unconnected-(U1-RX7-Pad28) -> Leg4 Coxa
- U1 pad 29: unconnected-(U1-TX7-Pad29) -> Leg5 Tibia
- U1 pad 3: unconnected-(U1-LRCLK2-Pad3) -> Leg3 Femur
- U1 pad 33: unconnected-(U1-MCLK2-Pad33) -> Leg5 Femur
- U1 pad 36: unconnected-(U1-CS2-Pad36) -> Leg5 Coxa
- U1 pad 37: unconnected-(U1-CS3-Pad37) -> Leg6 Tibia
- U1 pad 4: unconnected-(U1-BCLK2-Pad4) -> Leg3 Tibia
- U1 pad 5: unconnected-(U1-IN2-Pad5) -> Leg2 Coxa
- U1 pad 5V: unconnected-(U1-Pad5V) -> +5V
- U1 pad 6: unconnected-(U1-OUT1D-Pad6) -> Leg2 Femur
- U1 pad 7: unconnected-(U1-RX2-Pad7) -> Leg2 Tibia
- U1 pad 8: unconnected-(U1-TX2-Pad8) -> Leg1 Coxa
- U1 pad 9: unconnected-(U1-OUT1C-Pad9) -> Leg1 Femur
- U1 pad GND1: Net-(U1-GND-PadGND1) -> GND
- U1 pad GND2: Net-(U1-GND-PadGND1) -> GND
- U1 pad GND3: Net-(U1-GND-PadGND1) -> GND
- U1 pad GND4: Net-(U1-GND-PadGND1) -> GND
- U1 pad GND5: Net-(U1-GND-PadGND1) -> GND
- U1 pad VIN: unconnected-(U1-PadVIN) -> Teensy VIN
Routing:
- added copper zone on F.Cu, net (none)
- added copper zone on B.Cu, net GND
Other:
- board outline added: 96.5 x 96.5 mm

Commit message: pcb 3d models
Parts:
- moved U3 2.84 mm to (145.8, 71.8)
Changed lines of the file:
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@@
     (pad "2" thru_hole circle (at 7.62 0 270) (size 2.4 2.4) (drill 1.6) (layers "*.Cu" "*.Mask")
       (net 43 "Net-(J2-Pad2)") (pinfunction "2") (pintype "passive") (solder_mask_margin 0.102))
-    (model "${KIPRJMOD}/Components/Terminal 2 Pin/TB005-762-02BE.step"
-      (offset (xyz 7.5 -8 0))
-      (scale (xyz 1 1 1))
-      (rotate (xyz -90 0 -90))
+    (model "${HEXAPOD}/TB005-762-02BE.step"
+      (offset (xyz 7.6 -7.9 0))
+      (scale (xyz 1 1 1))
+      (rotate (xyz 90 180 90))
     )
   )
@@
       (net 42 "+BATT") (pinfunction "2") (pintype "passive") (solder_mask_margin 0.102))
     (model "${HEXAPOD}/TB005-762-02BE.step"
-      (offset (xyz 7.5 -8 0))
-      (scale (xyz 1 1 1))
-      (rotate (xyz -90 0 -90))
+      (offset (xyz 7.6 -7.9 0))
+      (scale (xyz 1 1 1))
+      (rotate (xyz 90 180 90))
     )
   )
@@
   )
   (footprint "RF_Module:nRF24L01_Breakout" (layer "F.Cu")
-    (at 147.02 69.305)
+    (at 145.75 71.845)
     (descr "nRF24L01 breakout board")
     (tags "nRF24L01 adapter breakout")
@@
     (pad "8" thru_hole circle (at 2.54 7.62) (size 1.7 1.7) (drill 1) (layers "*.Cu" "*.Mask")
       (net 60 "unconnected-(U3-IRQ-Pad8)") (pinfunction "IRQ") (pintype "output"))
-    (model "${KICAD6_3DMODEL_DIR}/RF_Module.3dshapes/nRF24L01_Breakout.wrl"
-      (offset (xyz 0 0 0))
-      (scale (xyz 1 1 1))
-      (rotate (xyz 0 0 0))
+    (model "${KIPRJMOD}/Components/nrf24l01/nRF24L01+.stp"
+      (offset (xyz 13 -5.5 1.5))
+      (scale (xyz 1 1 1))
+      (rotate (xyz -90 0 0))
     )
   )
@@
         (effects (font (size 1 1) (thickness 0.1)) (justify right bottom))
     )
+    (fp_text user "In+" (at 0.508 4.572 unlocked) (layer "F.SilkS")
+        (effects (font (size 1 1) (thickness 0.1)) (justify left bottom))
+    )
+    (fp_text user "In-" (at 0.508 19.304 unlocked) (layer "F.SilkS")
+        (effects (font (size 1 1) (thickness 0.1)) (justify left bottom))
+    )
     (fp_text user "Out-" (at 44.704 19.304 unlocked) (layer "F.SilkS")
         (effects (font (size 1 1) (thickness 0.1)) (justify right bottom))
     )
-    (fp_text user "In-" (at 0.508 19.304 unlocked) (layer "F.SilkS")
-        (effects (font (size 1 1) (thickness 0.1)) (justify left bottom))
-    )
-    (fp_text user "In+" (at 0.508 4.572 unlocked) (layer "F.SilkS")
-        (effects (font (size 1 1) (thickness 0.1)) (justify left bottom))
-    )
     (fp_text user "${REFERENCE}" (at 24.13 27.94 unlocked) (layer "F.Fab")
         (effects (font (size 1 1) (thickness 0.15)))
     )
-    (fp_rect (start 0 0) (end 45 23)
+    (fp_rect (start 0 0) (end 43.5 21.5)
       (stroke (width 0.1) (type solid)) (fill none) (layer "F.SilkS"))
-    (pad "1" thru_hole rect (at 1.778 1.778) (size 3 3) (drill 1.5) (layers "*.Cu" "*.Mask")
+    (pad "1" thru_hole rect (at 2 2.3) (size 3 3) (drill 1.5) (layers "*.Cu" "*.Mask")
       (net 42 "+BATT") (pinfunction "In+") (pintype "power_in"))
-    (pad "2" thru_hole rect (at 1.778 21.082) (size 3 3) (drill 1.5) (layers "*.Cu" "*.Mask")
+    (pad "2" thru_hole rect (at 2 19) (size 3 3) (drill 1.5) (layers "*.Cu" "*.Mask")
       (net 38 "GND") (pinfunction "In-") (pintype "power_in"))
-    (pad "3" thru_hole rect (at 43.18 1.778) (size 3 3) (drill 1.5) (layers "*.Cu" "*.Mask")
+    (pad "3" thru_hole rect (at 41.5 2.3) (size 3 3) (drill 1.5) (layers "*.Cu" "*.Mask")
       (net 59 "Teensy VIN") (pinfunction "Out+") (pintype "power_out"))
-    (pad "4" thru_hole rect (at 43.18 21.082) (size 3 3) (drill 1.5) (layers "*.Cu" "*.Mask")
+    (pad "4" thru_hole rect (at 41.5 19) (size 3 3) (drill 1.5) (layers "*.Cu" "*.Mask")
       (net 38 "GND") (pinfunction "Out-") (pintype "power_out"))
+    (model "${KIPRJMOD}/Components/Voltage Regulator LM2596/HW-411.STEP"
+      (offset (xyz 0 -0.5 0))
+      (scale (xyz 1 1 1))
+      (rotate (xyz -90 0 90))
+    )
   )
   (footprint "Connector_PinHeader_2.54mm:PinHeader_1x03_P2.54mm_Vertical" (layer "B.Cu")
@@
         (effects (font (size 1 1) (thickness 0.15)) (justify mirror))
     )
+    (fp_text user "SCL" (at -5.334 16.002 270 unlocked) (layer "B.SilkS")
+        (effects (font (size 1 1) (thickness 0.1)) (justify left bottom mirror))
+    )
+    (fp_text user "XCL" (at -5.334 8.382 270 unlocked) (layer "B.SilkS")
+        (effects (font (size 1 1) (thickness 0.1)) (justify left bottom mirror))
+    )
+    (fp_text user "INT" (at -5.334 3.302 270 unlocked) (layer "B.SilkS")
+        (effects (font (size 1 1) (thickness 0.1)) (justify left bottom mirror))
+    )
+    (fp_text user "SDA" (at -5.334 13.462 270 unlocked) (layer "B.SilkS")
+        (effects (font (size 1 1) (thickness 0.1)) (justify left bottom mirror))
+    )
     (fp_text user "XDA" (at -5.334 10.922 270 unlocked) (layer "B.SilkS")
         (effects (font (size 1 1) (thickness 0.1)) (justify left bottom mirror))
@@
         (effects (font (size 1 1) (thickness 0.1)) (justify left bottom mirror))
     )
-    (fp_text user "INT" (at -5.334 3.302 270 unlocked) (layer "B.SilkS")
-        (effects (font (size 1 1) (thickness 0.1)) (justify left bottom mirror))
-    )
-    (fp_text user "VCC" (at -5.334 21.082 270 unlocked) (layer "B.SilkS")
-        (effects (font (size 1 1) (thickness 0.1)) (justify left bottom mirror))
-    )
-    (fp_text user "SCL" (at -5.334 16.002 270 unlocked) (layer "B.SilkS")
-        (effects (font (size 1 1) (thickness 0.1)) (justify left bottom mirror))
-    )
-    (fp_text user "SDA" (at -5.334 13.462 270 unlocked) (layer "B.SilkS")
-        (effects (font (size 1 1) (thickness 0.1)) (justify left bottom mirror))
-    )
     (fp_text user "GND" (at -5.334 18.542 270 unlocked) (layer "B.SilkS")
         (effects (font (size 1 1) (thickness 0.1)) (justify left bottom mirror))
     )
-    (fp_text user "XCL" (at -5.334 8.382 270 unlocked) (layer "B.SilkS")
+    (fp_text user "VCC" (at -5.334 21.082 270 unlocked) (layer "B.SilkS")
         (effects (font (size 1 1) (thickness 0.1)) (justify left bottom mirror))
     )
@@
     (pad "8" thru_hole circle (at -6.222 3.81) (size 1.5 1.5) (drill 0.8) (layers "*.Cu" "*.Mask")
       (net 64 "unconnected-(U4-INT-Pad8)") (pinfunction "INT") (pintype "output"))
+    (model "${KIPRJMOD}/Components/MPU6050 THT/MPU6050.stp"
+      (offset (xyz -16.1 5.55 -7.5))
+      (scale (xyz 1 1 1))
+      (rotate (xyz -90 0 -90))
+    )
   )
   (footprint "Connector_PinHeader_2.54mm:PinHeader_1x03_P2.54mm_Vertical" (layer "B.Cu")
@@
     )
     (stroke (width 0.2) (type solid)) (fill none) (layer "Edge.Cuts"))
-  (dimension (type aligned) (layer "B.Cu")
-    (pts (xy 143.51 149.86) (xy 137.16 149.86))
-    (height -5.08)
-    (gr_text "6.3500 mm" (at 140.335 153.14) (layer "B.Cu")
-      (effects (font (size 1.5 1.5) (thickness 0.3)))
-    )
-    (format (prefix "") (suffix "") (units 3) (units_format 1) (precision 4))
-    (style (thickness 0.2) (arrow_length 1.27) (text_position_mode 0) (extension_height 0.58642) (extension_offset 0.5) keep_text_aligned)
-  )
-  (dimension (type aligned) (layer "B.Cu")
-    (pts (xy 179.07 125.73) (xy 175.26 130.81))
-    (height -9.990798)
-    (gr_text "6.3500 mm" (at 183.717638 133.184479 53.13010235) (layer "B.Cu")
-      (effects (font (size 1.5 1.5) (thickness 0.3)))
-    )
-    (format (prefix "") (suffix "") (units 3) (units_format 1) (precision 4))
-    (style (thickness 0.2) (arrow_length 1.27) (text_position_mode 0) (extension_height 0.58642) (extension_offset 0.5) keep_text_aligned)
-  )
-  (dimension (type aligned) (layer "B.Cu")
-    (pts (xy 143.51 149.86) (xy 149.86 149.86))
-    (height 5.08)
-    (gr_text "6.3500 mm" (at 146.685 153.14) (layer "B.Cu")
-      (effects (font (size 1.5 1.5) (thickness 0.3)))
-    )
-    (format (prefix "") (suffix "") (units 3) (units_format 1) (precision 4))
-    (style (thickness 0.2) (arrow_length 1.27) (text_position_mode 0) (extension_height 0.58642) (extension_offset 0.5) keep_text_aligned)
-  )
-  (dimension (type aligned) (layer "B.Cu")
-    (pts (xy 179.07 125.73) (xy 182.88 120.65))
-    (height 10.007992)
-    (gr_text "6.3500 mm" (at 187.541394 128.114795 53.13010235) (layer "B.Cu")
-      (effects (font (size 1.5 1.5) (thickness 0.3)))
-    )
-    (format (prefix "") (suffix "") (units 3) (units_format 1) (precision 4))
-    (style (thickness 0.2) (arrow_length 1.27) (text_position_mode 0) (extension_height 0.58642) (extension_offset 0.5) keep_text_aligned)
-  )
   (zone (net 0) (net_name "") (layer "F.Cu") (hatch edge 0.5)
     (connect_pads (clearance 0.5))

Commit message: traces
Parts:
- removed U2: Voltage Regulator, Voltage Regulator LM2596:Voltage Regulator LM2596
- added B1: Conn_01x01, Connector_PinHeader_2.54mm:PinHeader_1x01_P2.54mm_Vertical, F.Cu at (125.7, 65.4)
- added B2: Conn_01x01, Connector_PinHeader_2.54mm:PinHeader_1x01_P2.54mm_Vertical, F.Cu at (129.5, 65.4)
- added B3: Conn_01x01, Connector_PinHeader_2.54mm:PinHeader_1x01_P2.54mm_Vertical, F.Cu at (133.3, 65.4)
- added B3.3V1: Conn_01x02, Connector_PinHeader_2.54mm:PinHeader_1x02_P2.54mm_Vertical, F.Cu at (154.3, 65.4)
- added B4: Conn_01x01, Connector_PinHeader_2.54mm:PinHeader_1x01_P2.54mm_Vertical, F.Cu at (137.2, 65.4)
- added B5: Conn_01x01, Connector_PinHeader_2.54mm:PinHeader_1x01_P2.54mm_Vertical, F.Cu at (141.0, 65.4)
- added B5V1: Conn_01x02, Connector_PinHeader_2.54mm:PinHeader_1x02_P2.54mm_Vertical, F.Cu at (158.1, 65.4)
- added B6: Conn_01x01, Connector_PinHeader_2.54mm:PinHeader_1x01_P2.54mm_Vertical, F.Cu at (144.8, 65.4)
- added B7: Conn_01x01, Connector_PinHeader_2.54mm:PinHeader_1x01_P2.54mm_Vertical, F.Cu at (148.6, 65.4)
- added BGND1: Conn_01x02, Connector_PinHeader_2.54mm:PinHeader_1x02_P2.54mm_Vertical, F.Cu at (161.9, 65.4)
- added D1: D_Zener, Diode_THT:D_T-1_P5.08mm_Horizontal, F.Cu at (151.1, 115.6)
- added FS1: Foot Switch 1, Connector_PinHeader_2.54mm:PinHeader_1x02_P2.54mm_Vertical, B.Cu at (110.5, 90.8)
- added FS2: Foot Switch 2, Connector_PinHeader_2.54mm:PinHeader_1x02_P2.54mm_Vertical, B.Cu at (110.5, 95.2)
- added FS3: Foot Switch 3, Connector_PinHeader_2.54mm:PinHeader_1x02_P2.54mm_Vertical, B.Cu at (110.5, 99.7)
- added FS4: Foot Switch 4, Connector_PinHeader_2.54mm:PinHeader_1x02_P2.54mm_Vertical, B.Cu at (175.9, 91.2)
- added FS5: Foot Switch 5, Connector_PinHeader_2.54mm:PinHeader_1x02_P2.54mm_Vertical, B.Cu at (175.9, 95.9)
- added FS6: Foot Switch 6, Connector_PinHeader_2.54mm:PinHeader_1x02_P2.54mm_Vertical, B.Cu at (175.9, 100.5)
- added G***: LOGO, LOGO, F.Cu at (172.4, 113.9)
- added U5: Buck Converter 5V MP1584EN, Buck Converter 5V MP1584EN:Buck Converter 5V MP1584EN, F.Cu at (169.6, 100.9)
- R1: value 10k -> R1
- R2: value 22k -> R2
- U4: value Gyro -> Gyro MPU6050; moved to F.Cu
- moved Tib4 89.6 mm to (189.2, 81.7), turned to 90 degrees
- moved Fem4 83.0 mm to (189.2, 86.4), turned to 90 degrees
- moved Cox4 76.5 mm to (189.2, 91.0), turned to 90 degrees
- moved Tib1 72.2 mm to (97.8, 91.0), turned to -90 degrees
- moved Tib3 69.8 mm to (97.8, 121.3), turned to -90 degrees
- moved Tib5 67.7 mm to (189.2, 97.0), turned to 90 degrees
- moved Tib2 67.6 mm to (97.8, 106.0), turned to -90 degrees
- moved Fem1 66.0 mm to (97.8, 86.4), turned to -90 degrees
- moved Fem3 63.5 mm to (97.8, 116.6), turned to -90 degrees
- moved Fem5 61.2 mm to (189.2, 101.6), turned to 90 degrees
- moved Fem2 61.0 mm to (97.8, 101.4), turned to -90 degrees
- moved H3 60.8 mm to (167.6, 137.2), turned to 90 degrees
- moved H4 60.8 mm to (167.6, 66.0), turned to 90 degrees
- moved H1 60.6 mm to (119.6, 137.2), turned to 90 degrees
- moved H2 60.6 mm to (119.6, 66.0), turned to 90 degrees
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- renumbered J18 to Cox1, J15 to Cox2, J12 to Cox3, J9 to Cox4, J6 to Cox5, J1 to Cox6, J19 to Fem1, J16 to Fem2, J13 to Fem3, J10 to Fem4, J7 to Fem5, J3 to Fem6, J2 to T1, J5 to T2, J20 to Tib1, J17 to Tib2, J14 to Tib3, J11 to Tib4, J8 to Tib5, J4 to Tib6
Connections:
- U1 pad 10: Leg1 Tibia -> Leg1 Coxa
- U1 pad 17: unconnected-(U1-A3-Pad17) -> B6
- U1 pad 2: Leg3 Coxa -> Leg3 Tibia
- U1 pad 20: unconnected-(U1-A6-Pad20) -> B7
- U1 pad 21: unconnected-(U1-A7-Pad21) -> FS6
- U1 pad 22: unconnected-(U1-A8-Pad22) -> FS5
- U1 pad 23: unconnected-(U1-A9-Pad23) -> FS4
- U1 pad 25: Leg4 Femur -> Leg5 Femur
- U1 pad 28: Leg4 Coxa -> Leg5 Coxa
- U1 pad 29: Leg5 Tibia -> Leg6 Tibia
- U1 pad 30: unconnected-(U1-CRX3-Pad30) -> B2
- U1 pad 31: unconnected-(U1-CTX3-Pad31) -> B1
- U1 pad 33: Leg5 Femur -> Leg4 Femur
- U1 pad 34: unconnected-(U1-RX8-Pad34) -> FS1
- U1 pad 35: unconnected-(U1-TX8-Pad35) -> FS2
- U1 pad 36: Leg5 Coxa -> Leg4 Coxa
- U1 pad 37: Leg6 Tibia -> Leg5 Tibia
- U1 pad 38: unconnected-(U1-A14-Pad38) -> FS3
- U1 pad 39: unconnected-(U1-A15-Pad39) -> B3
- U1 pad 4: Leg3 Tibia -> Leg3 Coxa
- U1 pad 40: unconnected-(U1-A16-Pad40) -> B4
- U1 pad 41: unconnected-(U1-A17-Pad41) -> B5
- U1 pad 5: Leg2 Coxa -> Leg2 Tibia
- U1 pad 7: Leg2 Tibia -> Leg2 Coxa
- U1 pad 8: Leg1 Coxa -> Leg1 Tibia
Routing:
- net +BATT: track 0.00 -> 386.3 mm
- net +3.3V: track 0.00 -> 128.2 mm
- net Leg1 Coxa: track 0.00 -> 77.2 mm
- net Leg4 Tibia: track 0.00 -> 76.4 mm
- net Leg1 Femur: track 0.00 -> 70.4 mm
- net Leg6 Femur: track 0.00 -> 66.0 mm
- net Leg6 Coxa: track 0.00 -> 64.0 mm
- net Leg1 Tibia: track 0.00 -> 63.9 mm
- net Leg4 Femur: track 0.00 -> 62.2 mm
- net Leg4 Coxa: track 0.00 -> 60.2 mm
- net MOSI: track 0.00 -> 57.6 mm
- net Teensy VIN: track 0.00 -> 57.3 mm
- net Leg5 Tibia: track 0.00 -> 56.4 mm
- net Leg2 Coxa: track 0.00 -> 56.2 mm
- net MISO: track 0.00 -> 54.5 mm
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Other:
- board size 96.5 x 96.5 mm -> 96.5 x 81.3 mm
- copper layers 2 -> 4
- board text added: "+"
- board text added: "-"
- board text added: "Aecert Robotics"
- board text added: "Aecert's"
- board text added: "Battery"
- board text added: "Designed By:"
- board text added: "Hexapod"
- board text added: "Leg 1"
- board text added: "Leg 2"
- board text added: "Leg 3"
- board text added: "Leg 4"
- board text added: "Leg 5"
- board text added: "Leg 6"
- board text added: "Manufactured By:"
- board text added: "PCBWay"
- board text added: "Switch"
- board text added: "aecertrobotics.com"
- board text added: "pcbway.com"

Commit message: pcb updates
Other:
- board text added: "V 1.00"
Changed lines of the file:
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@@
     (effects (font (size 2 2) (thickness 0.3) bold) (justify bottom))
+  )
+  (gr_text "V 1.00" (at 176.53 75.565) (layer "F.SilkS")
+    (effects (font (size 1.5 1.5) (thickness 0.3) bold) (justify left bottom))
   )
   (gr_text "-" (at 123.82072 139.804125) (layer "F.SilkS")

Commit message: breakout updates
Parts:
- removed the B2 at (129.5, 65.4)
- removed the B3 at (133.3, 65.4)
- removed the B4 at (137.2, 65.4)
- removed B5, B6, B7: Conn_01x01, Connector_PinHeader_2.54mm:PinHeader_1x01_P2.54mm_Vertical
- B1: value Conn_01x01 -> Breakouts; footprint Connector_PinHeader_2.54mm:PinHeader_1x01_P2.54mm_Vertical -> Connector_PinSocket_2.54mm:PinSocket_1x07_P2.54mm_Vertical
- B2: renamed from BGND1; value Conn_01x02 -> GND; footprint Connector_PinHeader_2.54mm:PinHeader_1x02_P2.54mm_Vertical -> Connector_PinSocket_2.54mm:PinSocket_1x02_P2.54mm_Vertical
- B3: renamed from B3.3V1; value Conn_01x02 -> 3.3V; footprint Connector_PinHeader_2.54mm:PinHeader_1x02_P2.54mm_Vertical -> Connector_PinSocket_2.54mm:PinSocket_1x02_P2.54mm_Vertical
- B4: renamed from B5V1; value Conn_01x02 -> 5V; footprint Connector_PinHeader_2.54mm:PinHeader_1x02_P2.54mm_Vertical -> Connector_PinSocket_2.54mm:PinSocket_1x02_P2.54mm_Vertical
- moved B2 10.8 mm to (151.1, 64.8)
- moved B4 3.24 mm to (161.3, 64.8)
- moved B3 2.01 mm to (156.2, 64.8)
- moved B1 0.90 mm to (125.1, 66.0), turned to 90 degrees
Routing:
- net B7: track 25.7 -> 29.6 mm
- net B6: track 24.1 -> 27.5 mm
- net Teensy VIN: track 57.3 -> 54.0 mm
- net B3: track 24.8 -> 22.1 mm
- net B2: track 12.2 -> 10.0 mm
- net B5: track 24.1 -> 22.1 mm
- net B4: track 23.6 -> 22.1 mm
- net +3.3V: track 128.2 -> 129.6 mm
- net B1: track 10.9 -> 10.0 mm
Other:
- board text added: "17"
- board text added: "20"
- board text added: "30"
- board text added: "31"
- board text added: "39"
- board text added: "40"
- board text added: "41"

Commit message: PCB V1 Finished
Routing:
- net +3.3V: track 129.6 -> 140.9 mm
- net Teensy VIN: track 54.0 -> 59.0 mm
- net Leg4 Femur: track 62.2 -> 65.5 mm
- net Leg6 Tibia: track 32.3 -> 34.0 mm
- net Leg6 Femur: track 66.0 -> 67.4 mm
- net Leg6 Coxa: track 64.0 -> 65.4 mm
- net B7: track 29.6 -> 30.7 mm
- net Leg5 Coxa: track 40.2 -> 41.2 mm
- net Leg5 Femur: track 52.1 -> 53.1 mm
- net +BATT: track 386.3 -> 385.5 mm
- net Battery Voltage Divider: track 43.0 -> 42.5 mm

Commit message: pcb v1.01
Parts:
- added D2: LD271, LED_THT:LED_D5.0mm_IRGrey, F.Cu at (146.1, 64.8)
- added R3: 470u, Resistor_THT:R_Axial_DIN0207_L6.3mm_D2.5mm_P7.62mm_Horizontal, F.Cu at (154.9, 115.6)
- moved D1 2.54 mm to (148.6, 115.6)
- moved B2 1.27 mm to (152.4, 64.8)
- moved B3 0.63 mm to (156.8, 64.8)
Routing:
- net Net-(D2-A): track 0.00 -> 51.9 mm
- net +3.3V: track 140.9 -> 163.9 mm
- net Teensy VIN: track 59.0 -> 49.5 mm
- net +BATT: track 385.5 -> 382.0 mm
- net Battery Voltage Divider: track 42.5 -> 41.0 mm
- net B7: track 30.7 -> 29.6 mm
- net GND: track 0.00 -> 0.67 mm, vias 2 -> 4
Other:
- board text added: "Bottom"
- board text added: "Power"
- board text added: "Top"
- board text added: "V 1.01"
- board text removed: "V 1.00"
