File: PCB/Hexapod PCB KiCad Project/Hexapod PCB KiCad Project.kicad_sch (KiCad schematic)
At the start: 1 part, among them IC1 TEENSY_4.1

Commit message: pcb updates
Parts:
- removed IC1: TEENSY_4.1, TEENSY_4.1:TEENSY41, symbol TEENSY_4.1:TEENSY_4.1
- added J1: Male Pin Header 1x3, Connector_PinHeader_2.54mm:PinHeader_1x03_P2.54mm_Vertical, symbol Connector:Conn_01x03_Socket
- added J2: Power Terminal, Terminal 2 Pin:CUI_TB005-762-02BE, symbol Terminal 2 Pin:TB005-762-02BE
- added U1: DEV-16771, TEENSY 4.1:MODULE_DEV-16771, symbol TEENSY 4.1:DEV-16771
Connections:
- new net: U1.3.3V_1 (3.3V), U1.3.3V_2 (3.3V), U1.3.3V_3 (3.3V)
- new net: U1.GND1 (GND), U1.GND2 (GND), U1.GND3 (GND), U1.GND4 (GND), U1.GND5 (GND)
- new net: U1.USB_GND1 (USB_GND), U1.USB_GND2 (USB_GND)
Changed lines of the file:
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@@
 (kicad_sch (version 20230121) (generator eeschema)
   (paper "A4")
-  (symbol (lib_id "TEENSY_4.1:TEENSY_4.1") (at 120.015 56.515 0) (unit 1)
+  (symbol (lib_id "Connector:Conn_01x03_Socket") (at 46.355 58.42 0) (unit 1)
+    (in_bom yes) (on_board yes) (dnp no)
+    (property "Reference" "J1" (at 48.26 57.15 0)
+      (effects (font (size 1.27 1.27)) (justify left))
+    )
+    (property "Value" "Male Pin Header 1x3" (at 48.26 59.69 0)
+      (effects (font (size 1.27 1.27)) (justify left))
+    )
+    (property "Footprint" "Connector_PinHeader_2.54mm:PinHeader_1x03_P2.54mm_Vertical" (at 46.355 58.42 0)
+      (effects (font (size 1.27 1.27)) hide)
+    )
+    (property "Datasheet" "~" (at 46.355 58.42 0)
+      (effects (font (size 1.27 1.27)) hide)
+    )
+    (pin "1")
+    (pin "2")
+    (pin "3")
+    (instances
+      (project "Hexapod PCB KiCad Project"
+        (path "/55308d4e-8005-4344-88fa-e9149757c1fd"
+          (reference "J1") (unit 1)
+        )
+      )
+    )
+  )
+  (symbol (lib_id "Terminal 2 Pin:TB005-762-02BE") (at 48.895 96.52 0) (unit 1)
     (in_bom yes) (on_board yes) (dnp no) (fields_autoplaced)
-    (property "Reference" "IC1" (at 146.685 49.53 0)
+    (property "Reference" "J2" (at 55.88 93.98 0)
+      (effects (font (size 1.27 1.27)) (justify left))
+    )
+    (property "Value" "Power Terminal" (at 55.88 96.52 0)
+      (effects (font (size 1.27 1.27)) (justify left))
+    )
+    (property "Footprint" "Terminal 2 Pin:CUI_TB005-762-02BE" (at 48.895 96.52 0)
+      (effects (font (size 1.27 1.27)) (justify bottom) hide)
+    )
+    (property "Datasheet" "" (at 48.895 96.52 0)
+      (effects (font (size 1.27 1.27)) hide)
+    )
+    (property "MF" "Same Sky" (at 48.895 96.52 0)
+      (effects (font (size 1.27 1.27)) (justify bottom) hide)
+    )
+    (property "Description" "\n                        \n                            2~24 Poles, Screw Type, Horizontal, 7.62 Pitch, 26~10 (AWG), Terminal Block Connector  \n                        \n" (at 48.895 96.52 0)
+      (effects (font (size 1.27 1.27)) (justify bottom) hide)
+    )
+    (property "Package" "None" (at 48.895 96.52 0)
+      (effects (font (size 1.27 1.27)) (justify bottom) hide)
+    )
+    (property "Price" "None" (at 48.895 96.52 0)
+      (effects (font (size 1.27 1.27)) (justify bottom) hide)
+    )
+    (property "Check_prices" "https://www.snapeda.com/parts/TB005-762-02BE/Same+Sky/view-part/?ref=eda" (at 48.895 96.52 0)
+      (effects (font (size 1.27 1.27)) (justify bottom) hide)
+    )
+    (property "STANDARD" "Manufacturer Recommendations" (at 48.895 96.52 0)
+      (effects (font (size 1.27 1.27)) (justify bottom) hide)
+    )
+    (property "SnapEDA_Link" "https://www.snapeda.com/parts/TB005-762-02BE/Same+Sky/view-part/?ref=snap" (at 48.895 96.52 0)
+      (effects (font (size 1.27 1.27)) (justify bottom) hide)
+    )
+    (property "MP" "TB005-762-02BE" (at 48.895 96.52 0)
+      (effects (font (size 1.27 1.27)) (justify bottom) hide)
+    )
+    (property "Availability" "In Stock" (at 48.895 96.52 0)
+      (effects (font (size 1.27 1.27)) (justify bottom) hide)
+    )
+    (property "MANUFACTURER" "CUI" (at 48.895 96.52 0)
+      (effects (font (size 1.27 1.27)) (justify bottom) hide)
+    )
+    (pin "1")
+    (pin "2")
+    (instances
+      (project "Hexapod PCB KiCad Project"
+        (path "/55308d4e-8005-4344-88fa-e9149757c1fd"
+          (reference "J2") (unit 1)
+        )
+      )
+    )
+  )
+  (symbol (lib_id "TEENSY 4.1:DEV-16771") (at 160.02 88.265 0) (unit 1)
+    (in_bom yes) (on_board yes) (dnp no) (fields_autoplaced)
+    (property "Reference" "U1" (at 160.02 33.02 0)
       (effects (font (size 1.27 1.27)))
     )
-    (property "Value" "TEENSY_4.1" (at 146.685 52.07 0)
+    (property "Value" "DEV-16771" (at 160.02 35.56 0)
       (effects (font (size 1.27 1.27)))
     )
-    (property "Footprint" "TEENSY_4.1:TEENSY41" (at 120.015 56.515 0)
-      (effects (font (size 1.27 1.27)) (justify bottom) hide)
-    )
-    (property "Datasheet" "" (at 120.015 56.515 0)
-      (effects (font (size 1.27 1.27)) hide)
-    )
-    (property "Manufacturer_Name" "PJRC" (at 120.015 56.515 0)
-      (effects (font (size 1.27 1.27)) (justify bottom) hide)
-    )
-    (property "MF" "PJRC" (at 120.015 56.515 0)
-      (effects (font (size 1.27 1.27)) (justify bottom) hide)
-    )
-    (property "Mouser_Price-Stock" "" (at 120.015 56.515 0)
-      (effects (font (size 1.27 1.27)) (justify bottom) hide)
-    )
-    (property "Description" "\n                        \n                            \n                        \n" (at 120.015 56.515 0)
-      (effects (font (size 1.27 1.27)) (justify bottom) hide)
-    )
-    (property "Mouser_Part_Number" "" (at 120.015 56.515 0)
-      (effects (font (size 1.27 1.27)) (justify bottom) hide)
-    )
-    (property "Price" "None" (at 120.015 56.515 0)
-      (effects (font (size 1.27 1.27)) (justify bottom) hide)
-    )
-    (property "Package" "None" (at 120.015 56.515 0)
-      (effects (font (size 1.27 1.27)) (justify bottom) hide)
-    )
-    (property "Check_prices" "https://www.snapeda.com/parts/Teensy%204.1/PJRC/view-part/?ref=eda" (at 120.015 56.515 0)
-      (effects (font (size 1.27 1.27)) (justify bottom) hide)
-    )
-    (property "Height" "mm" (at 120.015 56.515 0)
-      (effects (font (size 1.27 1.27)) (justify bottom) hide)
-    )
-    (property "MP" "Teensy 4.1" (at 120.015 56.515 0)
-      (effects (font (size 1.27 1.27)) (justify bottom) hide)
-    )
-    (property "SnapEDA_Link" "https://www.snapeda.com/parts/Teensy%204.1/PJRC/view-part/?ref=snap" (at 120.015 56.515 0)
-      (effects (font (size 1.27 1.27)) (justify bottom) hide)
-    )
-    (property "Arrow_Price-Stock" "" (at 120.015 56.515 0)
-      (effects (font (size 1.27 1.27)) (justify bottom) hide)
-    )
-    (property "Arrow_Part_Number" "" (at 120.015 56.515 0)
-      (effects (font (size 1.27 1.27)) (justify bottom) hide)
-    )
-    (property "Availability" "Not in stock" (at 120.015 56.515 0)
-      (effects (font (size 1.27 1.27)) (justify bottom) hide)
-    )
-    (property "Manufacturer_Part_Number" "TEENSY 4.1" (at 120.015 56.515 0)
-      (effects (font (size 1.27 1.27)) (justify bottom) hide)
-    )
+    (property "Footprint" "TEENSY 4.1:MODULE_DEV-16771" (at 160.02 88.265 0)
+      (effects (font (size 1.27 1.27)) (justify bottom) hide)
+    )
+    (property "Datasheet" "" (at 160.02 88.265 0)
+      (effects (font (size 1.27 1.27)) hide)
+    )
+    (property "MF" "SparkFun Electronics" (at 160.02 88.265 0)
+      (effects (font (size 1.27 1.27)) (justify bottom) hide)
+    )
+    (property "MAXIMUM_PACKAGE_HEIGHT" "4.07mm" (at 160.02 88.265 0)
+      (effects (font (size 1.27 1.27)) (justify bottom) hide)
+    )
+    (property "Package" "None" (at 160.02 88.265 0)
+      (effects (font (size 1.27 1.27)) (justify bottom) hide)
+    )
+    (property "Price" "None" (at 160.02 88.265 0)
+      (effects (font (size 1.27 1.27)) (justify bottom) hide)
+    )
+    (property "Check_prices" "https://www.snapeda.com/parts/DEV-16771/SparkFun/view-part/?ref=eda" (at 160.02 88.265 0)
+      (effects (font (size 1.27 1.27)) (justify bottom) hide)
+    )
+    (property "STANDARD" "Manufacturer recommendations" (at 160.02 88.265 0)
+      (effects (font (size 1.27 1.27)) (justify bottom) hide)
+    )
+    (property "PARTREV" "4.1" (at 160.02 88.265 0)
+      (effects (font (size 1.27 1.27)) (justify bottom) hide)
+    )
+    (property "SnapEDA_Link" "https://www.snapeda.com/parts/DEV-16771/SparkFun/view-part/?ref=snap" (at 160.02 88.265 0)
+      (effects (font (size 1.27 1.27)) (justify bottom) hide)
+    )
+    (property "MP" "DEV-16771" (at 160.02 88.265 0)
+      (effects (font (size 1.27 1.27)) (justify bottom) hide)
+    )
+    (property "Description" "\n                        \n                            RT1062 Teensy 4.1 series ARM® Cortex®-M7 MPU Embedded Evaluation Board\n                        \n" (at 160.02 88.265 0)
+      (effects (font (size 1.27 1.27)) (justify bottom) hide)
+    )
+    (property "Availability" "In Stock" (at 160.02 88.265 0)
+      (effects (font (size 1.27 1.27)) (justify bottom) hide)
+    )
+    (property "MANUFACTURER" "SparkFun Electronics" (at 160.02 88.265 0)
+      (effects (font (size 1.27 1.27)) (justify bottom) hide)
+    )
+    (pin "0")
     (pin "1")
     (pin "10")
@@
     (pin "29")
     (pin "3")
+    (pin "3.3V_1")
+    (pin "3.3V_2")
+    (pin "3.3V_3")
     (pin "30")
     (pin "31")
@@
     (pin "40")
     (pin "41")
-    (pin "42")
-    (pin "43")
-    (pin "44")
-    (pin "45")
-    (pin "46")
-    (pin "47")
-    (pin "48")
-    (pin "49")
     (pin "5")
-    (pin "50")
-    (pin "51")
-    (pin "52")
-    (pin "53")
-    (pin "55")
-    (pin "57")
+    (pin "5V")
     (pin "6")
-    (pin "68")
-    (pin "69")
     (pin "7")
-    (pin "70")
-    (pin "71")
     (pin "8")
     (pin "9")
+    (pin "D+")
+    (pin "D-")
+    (pin "GND1")
+    (pin "GND2")
+    (pin "GND3")
+    (pin "GND4")
+    (pin "GND5")
+    (pin "LED")
+    (pin "ON/OFF")
+    (pin "PROGRAM")
+    (pin "R+")
+    (pin "R-")
+    (pin "T+")
+    (pin "T-")
+    (pin "USB_GND1")
+    (pin "USB_GND2")
+    (pin "VBAT")
+    (pin "VIN")
+    (pin "VUSB")
     (instances
       (project "Hexapod PCB KiCad Project"
         (path "/55308d4e-8005-4344-88fa-e9149757c1fd"
-          (reference "IC1") (unit 1)
+          (reference "U1") (unit 1)
         )
       )

Commit message: Pcb updates
Parts:
- removed J1: Male Pin Header 1x3, Connector_PinHeader_2.54mm:PinHeader_1x03_P2.54mm_Vertical, symbol Connector:Conn_01x03_Socket
- removed J2: Power Terminal, Terminal 2 Pin:CUI_TB005-762-02BE, symbol Terminal 2 Pin:TB005-762-02BE
- removed U1: DEV-16771, TEENSY 4.1:MODULE_DEV-16771, symbol TEENSY 4.1:DEV-16771
- added C1: 50V 10uF, Capacitor_THT:CP_Radial_D5.0mm_P2.00mm, symbol Device:C_Polarized
- added C2: 50V 0.1uF, Capacitor_THT:CP_Radial_D4.0mm_P2.00mm, symbol Device:C_Polarized
- added C3, C4: 16V 1000uf, Capacitor_THT:CP_Radial_D10.0mm_P5.00mm, symbol Device:C_Polarized
- added H1, H2, H3, H4: MountingHole, MountingHole:MountingHole_3.2mm_M3, symbol Mechanical:MountingHole
- added J2: Battery, Terminal 2 Pin:CUI_TB005-762-02BE, symbol Power Terminal 2 Pin:TB005-762-02BE
- added J5: Switch, Terminal 2 Pin:CUI_TB005-762-02BE, symbol Power Terminal 2 Pin:TB005-762-02BE
- added R1: 10k, Resistor_THT:R_Axial_DIN0207_L6.3mm_D2.5mm_P7.62mm_Horizontal, symbol Device:R
- added R2: 22k, Resistor_THT:R_Axial_DIN0207_L6.3mm_D2.5mm_P7.62mm_Horizontal, symbol Device:R
- added U1: DEV-16771, Teensy 4.1:MODULE_DEV-16771, symbol Teensy 4.1:DEV-16771
- added U2: Voltage Regulator, Voltage Regulator LM2596:Voltage Regulator LM2596, symbol Voltage Regulator LM2596:Voltage_Regulator_LM2596
- added U3: NRF24L01_Breakout, RF_Module:nRF24L01_Breakout, symbol RF:NRF24L01_Breakout
- added U4: Gyro, MPU6050 THT:MPU6050 THT, symbol MPU6050 THT:MPU6050_THT
Connections:
- new net: U1.USB_GND1 (USB_GND), U1.USB_GND2 (USB_GND)
- new net: J2.2, J5.1
- new net +3.3V: C1.1, C2.1, U1.3.3V_1 (3.3V), U1.3.3V_2 (3.3V), U1.3.3V_3 (3.3V), U3.2 (VCC), U4.1 (VCC)
- new net +5V: U1.5V
- new net +BATT: C3.1, C4.1, J5.2, R1.1, U2.1 (In+)
- new net Battery Voltage Divider: R1.2, R2.1, U1.16 (A2)
- new net CE: U1.26 (A12), U3.3 (CE)
- new net CSN: U1.27 (A13), U3.4 (~{CSN})
- new net GND: C1.2, C2.2, C3.2, C4.2, J2.1, R2.2, U1.GND1 (GND), U1.GND2 (GND), U1.GND3 (GND), U1.GND4 (GND), U1.GND5 (GND), U2.2 (In-), U2.4 (Out-), U3.1 (GND), U4.2 (GND)
- new net Gyro SCL: U1.19 (A5), U4.3 (SCL)
- new net Gyro SDA: U1.18 (A4), U4.4 (SDA)
- new net Leg1 Coxa: U1.8 (TX2)
- new net Leg1 Femur: U1.9 (OUT1C)
- new net Leg1 Tibia: U1.10 (CS1)
- new net Leg2 Coxa: U1.5 (IN2)
- new net Leg2 Femur: U1.6 (OUT1D)
- new net Leg2 Tibia: U1.7 (RX2)
- new net Leg3 Coxa: U1.2 (OUT2)
- new net Leg3 Femur: U1.3 (LRCLK2)
- new net Leg3 Tibia: U1.4 (BCLK2)
- new net Leg4 Coxa: U1.28 (RX7)
- new net Leg4 Femur: U1.25 (A11)
- new net Leg4 Tibia: U1.24 (A10)
- new net Leg5 Coxa: U1.36 (CS2)
- new net Leg5 Femur: U1.33 (MCLK2)
- new net Leg5 Tibia: U1.29 (TX7)
- new net Leg6 Coxa: U1.15 (A1)
- new net Leg6 Femur: U1.14 (A0)
- new net Leg6 Tibia: U1.37 (CS3)
- new net MISO: U1.12 (MISO), U3.7 (MISO)
- new net MOSI: U1.11 (MOSI), U3.6 (MOSI)
- new net SCK: U1.13 (SCK), U3.5 (SCK)
- new net Teensy VIN: U1.VIN, U2.3 (Out+)
- no-connect marks 0 -> 2
Other:
- added sheet Leg 1 (Leg.kicad_sch)
- added sheet Leg 2 (Leg.kicad_sch)
- added sheet Leg 3 (Leg.kicad_sch)
- added sheet Leg 4 (Leg.kicad_sch)
- added sheet Leg 5 (Leg.kicad_sch)
- added sheet Leg 6 (Leg.kicad_sch)
- note added: "Gyro"
- note added: "Mounting Holes"
- note added: "NRF"
- note added: "Power"
- note added: "Servos"
- note added: "Teensy 4.1"

Commit message: sheet data
Other:
- company: (none) -> Aecert Robotics
- title: (none) -> Hexapod PCB - Teensy 4.1
- moved on the sheet: U1

Commit message: traces
Parts:
- removed U2: Voltage Regulator, Voltage Regulator LM2596:Voltage Regulator LM2596, symbol Voltage Regulator LM2596:Voltage_Regulator_LM2596
- added B1, B2, B3, B4, B5, B6, B7: Conn_01x01, Connector_PinHeader_2.54mm:PinHeader_1x01_P2.54mm_Vertical, symbol Connector_Generic:Conn_01x01
- added B3.3V1, B5V1, BGND1: Conn_01x02, Connector_PinHeader_2.54mm:PinHeader_1x02_P2.54mm_Vertical, symbol Connector_Generic:Conn_01x02
- added D1: D_Zener, Diode_THT:D_T-1_P5.08mm_Horizontal, symbol Device:D_Zener
- added FS1: Foot Switch 1, Connector_PinHeader_2.54mm:PinHeader_1x02_P2.54mm_Vertical, symbol Connector_Generic:Conn_01x02
- added FS2: Foot Switch 2, Connector_PinHeader_2.54mm:PinHeader_1x02_P2.54mm_Vertical, symbol Connector_Generic:Conn_01x02
- added FS3: Foot Switch 3, Connector_PinHeader_2.54mm:PinHeader_1x02_P2.54mm_Vertical, symbol Connector_Generic:Conn_01x02
- added FS4: Foot Switch 4, Connector_PinHeader_2.54mm:PinHeader_1x02_P2.54mm_Vertical, symbol Connector_Generic:Conn_01x02
- added FS5: Foot Switch 5, Connector_PinHeader_2.54mm:PinHeader_1x02_P2.54mm_Vertical, symbol Connector_Generic:Conn_01x02
- added FS6: Foot Switch 6, Connector_PinHeader_2.54mm:PinHeader_1x02_P2.54mm_Vertical, symbol Connector_Generic:Conn_01x02
- added U5: Buck Converter 5V MP1584EN, Buck Converter 5V MP1584EN:Buck Converter 5V MP1584EN, symbol Buck Converter 5v MP1584EN:Buck_Converter_5v_MP1584EN
- R1: value 10k -> R1
- R2: value 22k -> R2
- U4: value Gyro -> Gyro MPU6050
- renumbered J2 to T1, J5 to T2
Connections:
- net +3.3V: now also B3.3V1.1 (Pin_1), B3.3V1.2 (Pin_2)
- net +BATT: now also U5.1 (In+)
- net Battery Voltage Divider: now also D1.1 (K)
- net GND: now also BGND1.1 (Pin_1), BGND1.2 (Pin_2), D1.2 (A), FS1.1 (Pin_1), FS2.1 (Pin_1), FS3.1 (Pin_1), FS4.1 (Pin_1), FS5.1 (Pin_1), FS6.1 (Pin_1), U5.2 (In-), U5.4 (Out-)
- net Leg1 Coxa: now also U1.10 (CS1); no longer U1.8 (TX2)
- net Leg1 Tibia: now also U1.8 (TX2); no longer U1.10 (CS1)
- net Leg2 Coxa: now also U1.7 (RX2); no longer U1.5 (IN2)
- net Leg2 Tibia: now also U1.5 (IN2); no longer U1.7 (RX2)
- net Leg3 Coxa: now also U1.4 (BCLK2); no longer U1.2 (OUT2)
- net Leg3 Tibia: now also U1.2 (OUT2); no longer U1.4 (BCLK2)
- net Leg4 Coxa: now also U1.36 (CS2); no longer U1.28 (RX7)
- net Leg4 Femur: now also U1.33 (MCLK2); no longer U1.25 (A11)
- net Leg5 Coxa: now also U1.28 (RX7); no longer U1.36 (CS2)
- net Leg5 Femur: now also U1.25 (A11); no longer U1.33 (MCLK2)
- net Leg5 Tibia: now also U1.37 (CS3); no longer U1.29 (TX7)
- net Leg6 Tibia: now also U1.29 (TX7); no longer U1.37 (CS3)
- net Teensy VIN: now also B5V1.1 (Pin_1), B5V1.2 (Pin_2), U5.3 (Out+)
- net B6: now reaches U1.17 (A3)
- net B6: now also B6.1 (Pin_1)
- net B7: now reaches U1.20 (A6)
- net B7: now also B7.1 (Pin_1)
- net FS6: now reaches U1.21 (A7)
- net FS6: now also FS6.2 (Pin_2)
- net FS5: now reaches U1.22 (A8)
- net FS5: now also FS5.2 (Pin_2)
- net FS4: now reaches U1.23 (A9)
- net FS4: now also FS4.2 (Pin_2)
- net B2: now reaches U1.30 (CRX3)
- net B2: now also B2.1 (Pin_1)
- net B1: now reaches U1.31 (CTX3)
- net B1: now also B1.1 (Pin_1)
- net FS1: now reaches U1.34 (RX8)
- net FS1: now also FS1.2 (Pin_2)
- net FS2: now reaches U1.35 (TX8)
- net FS2: now also FS2.2 (Pin_2)
- net FS3: now reaches U1.38 (A14)
- net FS3: now also FS3.2 (Pin_2)
- net B3: now reaches U1.39 (A15)
- net B3: now also B3.1 (Pin_1)
- net B4: now reaches U1.40 (A16)
- net B4: now also B4.1 (Pin_1)
- net B5: now reaches U1.41 (A17)
- net B5: now also B5.1 (Pin_1)
Other:
- note added: "Breakouts"
- note added: "Foot Switches"
- moved on the sheet: C1, C2, C3, C4, R1, R2, T1, T2, U1, U3

Commit message: breakout updates
Parts:
- removed B2, B3, B4, B5, B6, B7: Conn_01x01, Connector_PinHeader_2.54mm:PinHeader_1x01_P2.54mm_Vertical, symbol Connector_Generic:Conn_01x01
- B1: value Conn_01x01 -> Breakouts; footprint Connector_PinHeader_2.54mm:PinHeader_1x01_P2.54mm_Vertical -> Connector_PinSocket_2.54mm:PinSocket_1x07_P2.54mm_Vertical; symbol Connector_Generic:Conn_01x01 -> Connector_Generic:Conn_01x07
- B2: renamed from BGND1; value Conn_01x02 -> GND; footprint Connector_PinHeader_2.54mm:PinHeader_1x02_P2.54mm_Vertical -> Connector_PinSocket_2.54mm:PinSocket_1x02_P2.54mm_Vertical
- B3: renamed from B3.3V1; value Conn_01x02 -> 3.3V; footprint Connector_PinHeader_2.54mm:PinHeader_1x02_P2.54mm_Vertical -> Connector_PinSocket_2.54mm:PinSocket_1x02_P2.54mm_Vertical
- B4: renamed from B5V1; value Conn_01x02 -> 5V; footprint Connector_PinHeader_2.54mm:PinHeader_1x02_P2.54mm_Vertical -> Connector_PinSocket_2.54mm:PinSocket_1x02_P2.54mm_Vertical
Connections:
- net B2: now also B1.2 (Pin_2)
- net B3: now also B1.3 (Pin_3)
- net B4: now also B1.4 (Pin_4)
- net B5: now also B1.5 (Pin_5)
- net B6: now also B1.6 (Pin_6)
- net B7: now also B1.7 (Pin_7)
Other:
- moved on the sheet: B2, B3, B4, C3, C4, D1, R1, R2, T1, T2, U5

Commit message: pcb v1.01
Parts:
- added D2: LD271, LED_THT:LED_D5.0mm_IRGrey, symbol LED:LD271
- added R3: 470u, Resistor_THT:R_Axial_DIN0207_L6.3mm_D2.5mm_P7.62mm_Horizontal, symbol Device:R
Connections:
- net +3.3V: now also R3.2
- net GND: now also D2.1 (K)
- new net: D2.2 (A), R3.1
Changed lines of the file:
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@@
+    (stroke (width 0) (type default))
+  )
+  (wire (pts (xy 117.475 36.195) (xy 118.745 36.195))
     (stroke (width 0) (type default))
   )
@@
   )
   (wire (pts (xy 43.815 36.83) (xy 48.895 36.83))
+    (stroke (width 0) (type default))
+  )
+  (wire (pts (xy 108.585 36.195) (xy 109.855 36.195))
     (stroke (width 0) (type default))
   )
@@
         (path "/55308d4e-8005-4344-88fa-e9149757c1fd"
           (reference "#PWR019") (unit 1)
+        )
+      )
+    )
+  )
+  (symbol (lib_id "power:+3.3V") (at 118.745 36.195 270) (unit 1)
+    (in_bom yes) (on_board yes) (dnp no) (fields_autoplaced)
+    (property "Reference" "#PWR035" (at 114.935 36.195 0)
+      (effects (font (size 1.27 1.27)) hide)
+    )
+    (property "Value" "+3.3V" (at 122.555 36.195 90)
+      (effects (font (size 1.27 1.27)) (justify left))
+    )
+    (property "Footprint" "" (at 118.745 36.195 0)
+      (effects (font (size 1.27 1.27)) hide)
+    )
+    (property "Datasheet" "" (at 118.745 36.195 0)
+      (effects (font (size 1.27 1.27)) hide)
+    )
+    (pin "1")
+    (instances
+      (project "Hexapod PCB KiCad Project"
+        (path "/55308d4e-8005-4344-88fa-e9149757c1fd"
+          (reference "#PWR035") (unit 1)
         )
       )
@@
     )
   )
+  (symbol (lib_id "Device:R") (at 113.665 36.195 90) (unit 1)
+    (in_bom yes) (on_board yes) (dnp no) (fields_autoplaced)
+    (property "Reference" "R3" (at 113.665 30.48 90)
+      (effects (font (size 1.27 1.27)))
+    )
+    (property "Value" "470u" (at 113.665 33.02 90)
+      (effects (font (size 1.27 1.27)))
+    )
+    (property "Footprint" "Resistor_THT:R_Axial_DIN0207_L6.3mm_D2.5mm_P7.62mm_Horizontal" (at 113.665 37.973 90)
+      (effects (font (size 1.27 1.27)) hide)
+    )
+    (property "Datasheet" "~" (at 113.665 36.195 0)
+      (effects (font (size 1.27 1.27)) hide)
+    )
+    (pin "1")
+    (pin "2")
+    (instances
+      (project "Hexapod PCB KiCad Project"
+        (path "/55308d4e-8005-4344-88fa-e9149757c1fd"
+          (reference "R3") (unit 1)
+        )
+      )
+    )
+  )
   (symbol (lib_id "Connector_Generic:Conn_01x02") (at 36.195 184.785 0) (unit 1)
     (in_bom yes) (on_board yes) (dnp no) (fields_autoplaced)
@@
     )
   )
+  (symbol (lib_id "LED:LD271") (at 106.045 36.195 0) (unit 1)
+    (in_bom yes) (on_board yes) (dnp no) (fields_autoplaced)
+    (property "Reference" "D2" (at 104.902 27.94 0)
+      (effects (font (size 1.27 1.27)))
+    )
+    (property "Value" "LD271" (at 104.902 30.48 0)
+      (effects (font (size 1.27 1.27)))
+    )
+    (property "Footprint" "LED_THT:LED_D5.0mm_IRGrey" (at 106.045 31.75 0)
+      (effects (font (size 1.27 1.27)) hide)
+    )
+    (property "Datasheet" "http://www.alliedelec.com/m/d/40788c34903a719969df15f1fbea1056.pdf" (at 104.775 36.195 0)
+      (effects (font (size 1.27 1.27)) hide)
+    )
+    (pin "1")
+    (pin "2")
+    (instances
+      (project "Hexapod PCB KiCad Project"
+        (path "/55308d4e-8005-4344-88fa-e9149757c1fd"
+          (reference "D2") (unit 1)
+        )
+      )
+    )
+  )
   (symbol (lib_id "power:GND") (at 31.115 184.785 270) (unit 1)
     (in_bom yes) (on_board yes) (dnp no) (fields_autoplaced)
@@
         )
       )
+    )
+  )
+  (symbol (lib_id "power:GND") (at 100.965 36.195 270) (unit 1)
+    (in_bom yes) (on_board yes) (dnp no) (fields_autoplaced)
+    (property "Reference" "#PWR036" (at 94.615 36.195 0)
+      (effects (font (size 1.27 1.27)) hide)
+    )
+    (property "Value" "GND" (at 97.79 36.195 90)
+      (effects (font (size 1.27 1.27)) (justify right))
+    )
+    (property "Footprint" "" (at 100.965 36.195 0)
+      (effects (font (size 1.27 1.27)) hide)
+    )
+    (property "Datasheet" "" (at 100.965 36.195 0)
+      (effects (font (size 1.27 1.27)) hide)
+    )
+    (pin "1")
+    (instances
+      (project "Hexapod PCB KiCad Project"
+        (path "/55308d4e-8005-4344-88fa-e9149757c1fd"
+          (reference "#PWR036") (unit 1)
+        )
+      )
